File: SE_DES_2/base_robot.sch (EAGLE design)
At the start: 12 parts

Commit message: pcb files for sen des se_des_2 is the latest one
Parts:
- added U$13: 3_4_BALLCASTER, 3_4_BALLCASTER:3_4_BALLCASTER
- added U$14, U$15: MOTOR_BRACKET_25D, MOTOR_BRACKET_25D:MOTOR_BRACKET_25D
Changed lines of the file:
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@@
 <part name="U$11" library="IMU" deviceset="IMU" device=""/>
 <part name="U$12" library="HC05_BLUETOOTH" deviceset="HC05_BLUETOOTH" device=""/>
+<part name="U$13" library="3_4_BALLCASTER" deviceset="3_4_BALLCASTER" device=""/>
+<part name="U$14" library="MOTOR_BRACKET_25D" deviceset="MOTOR_BRACKET_25D" device=""/>
+<part name="U$15" library="MOTOR_BRACKET_25D" deviceset="MOTOR_BRACKET_25D" device=""/>
 </parts>
 <sheets>
@@
 <instance part="U$11" gate="G$1" x="144.78" y="81.28" smashed="yes"/>
 <instance part="U$12" gate="G$1" x="93.98" y="96.52" smashed="yes"/>
+<instance part="U$13" gate="G$1" x="248.92" y="91.44" smashed="yes"/>
+<instance part="U$14" gate="G$1" x="116.84" y="-15.24" smashed="yes"/>
+<instance part="U$15" gate="G$1" x="193.04" y="-15.24" smashed="yes"/>
 </instances>
 <busses>
